Commit message: Backing up work

File: box_pendulum/resources/cubebot_3D.urdf (robot description, URDF)
Before this commit: robot cubebot, 15 links, 14 joints
Links:
- removed link corner1
- removed link corner2
- removed link corner3
- removed link corner4
- removed link corner5
- removed link corner6
- removed link corner7
- removed link corner8
- removed link cube
- removed link wheel10
- removed link wheel11
- removed link wheel20
- removed link wheel21
- removed link wheel30
- removed link wheel31
- added link CornerBumper_1, mass 0.01; collision sphere radius=0.03; visual sphere radius=0.03
- added link CornerBumper_2, mass 0.01; collision sphere radius=0.03; visual sphere radius=0.03
- added link CornerBumper_3, mass 0.01; collision sphere radius=0.03; visual sphere radius=0.03
- added link CornerBumper_4, mass 0.01; collision sphere radius=0.03; visual sphere radius=0.03
- added link CornerBumper_5, mass 0.01; collision sphere radius=0.03; visual sphere radius=0.03
- added link CornerBumper_6, mass 0.01; collision sphere radius=0.03; visual sphere radius=0.03
- added link CornerBumper_7, mass 0.01; collision sphere radius=0.03; visual sphere radius=0.03
- added link CornerBumper_8, mass 0.01; collision sphere radius=0.03; visual sphere radius=0.03
- added link CubeBody, mass 0.1; collision box size=0.3 0.3 0.3; visual box size=0.3 0.3 0.3
- added link InertialWheel_1, mass 0.1; visual cylinder length=0.01 radius=0.08
- added link InertialWheel_2, mass 0.1; visual cylinder length=0.01 radius=0.08
- added link InertialWheel_3, mass 0.1; visual cylinder length=0.01 radius=0.08
- added link InertialWheel_4, mass 0.1; visual cylinder length=0.01 radius=0.08
- added link InertialWheel_5, mass 0.1; visual cylinder length=0.01 radius=0.08
- added link InertialWheel_6, mass 0.1; visual cylinder length=0.01 radius=0.08
Joints:
- removed joint cube corner1
- removed joint cube corner2
- removed joint cube corner3
- removed joint cube corner4
- removed joint cube corner5
- removed joint cube corner6
- removed joint cube corner7
- removed joint cube corner8
- removed joint cube to wheel10
- removed joint cube to wheel11
- removed joint cube to wheel20
- removed joint cube to wheel21
- removed joint cube to wheel30
- removed joint cube to wheel31
- added joint $continuous_CubeBody_InertialWheel_1: type continuous, parent CubeBody, child InertialWheel_1, origin xyz=0.15 0 0 rpy=0 1.57075 0, axis 0 0 1
- added joint $continuous_CubeBody_InertialWheel_2: type continuous, parent CubeBody, child InertialWheel_2, origin xyz=-0.15 0 0 rpy=0 1.57075 0, axis 0 0 1
- added joint $continuous_CubeBody_InertialWheel_3: type continuous, parent CubeBody, child InertialWheel_3, origin xyz=0 0.15 0 rpy=1.57075 0 0, axis 0 0 1
- added joint $continuous_CubeBody_InertialWheel_4: type continuous, parent CubeBody, child InertialWheel_4, origin xyz=0 -0.15 0 rpy=1.57075 0 0, axis 0 0 1
- added joint $continuous_CubeBody_InertialWheel_5: type continuous, parent CubeBody, child InertialWheel_5, origin xyz=0 0 0.15 rpy=0 0 1.57075, axis 0 0 1
- added joint $continuous_CubeBody_InertialWheel_6: type continuous, parent CubeBody, child InertialWheel_6, origin xyz=0 0 -0.15 rpy=0 0 1.57075, axis 0 0 1
- added joint $fixed_CubeBody_CornerBumper_1: type fixed, parent CubeBody, child CornerBumper_1, origin xyz=0.15 0.15 0.15 rpy=0 0 0
- added joint $fixed_CubeBody_CornerBumper_2: type fixed, parent CubeBody, child CornerBumper_2, origin xyz=-0.15 0.15 0.15 rpy=0 0 0
- added joint $fixed_CubeBody_CornerBumper_3: type fixed, parent CubeBody, child CornerBumper_3, origin xyz=0.15 -0.15 0.15 rpy=0 0 0
- added joint $fixed_CubeBody_CornerBumper_4: type fixed, parent CubeBody, child CornerBumper_4, origin xyz=-0.15 -0.15 0.15 rpy=0 0 0
- added joint $fixed_CubeBody_CornerBumper_5: type fixed, parent CubeBody, child CornerBumper_5, origin xyz=0.15 0.15 -0.15 rpy=0 0 0
- added joint $fixed_CubeBody_CornerBumper_6: type fixed, parent CubeBody, child CornerBumper_6, origin xyz=-0.15 0.15 -0.15 rpy=0 0 0
- added joint $fixed_CubeBody_CornerBumper_7: type fixed, parent CubeBody, child CornerBumper_7, origin xyz=0.15 -0.15 -0.15 rpy=0 0 0
- added joint $fixed_CubeBody_CornerBumper_8: type fixed, parent CubeBody, child CornerBumper_8, origin xyz=-0.15 -0.15 -0.15 rpy=0 0 0

File: xacro/test.urdf (robot description, URDF)
Before this commit: robot test, 1 links, 0 joints
Links:
- removed link base_link
- added link CornerBumper_1, mass 0.01; collision sphere radius=0.03; visual sphere radius=0.03
- added link CornerBumper_2, mass 0.01; collision sphere radius=0.03; visual sphere radius=0.03
- added link CornerBumper_3, mass 0.01; collision sphere radius=0.03; visual sphere radius=0.03
- added link CornerBumper_4, mass 0.01; collision sphere radius=0.03; visual sphere radius=0.03
- added link CornerBumper_5, mass 0.01; collision sphere radius=0.03; visual sphere radius=0.03
- added link CornerBumper_6, mass 0.01; collision sphere radius=0.03; visual sphere radius=0.03
- added link CornerBumper_7, mass 0.01; collision sphere radius=0.03; visual sphere radius=0.03
- added link CornerBumper_8, mass 0.01; collision sphere radius=0.03; visual sphere radius=0.03
- added link CubeBody, mass 0.1; collision box size=0.3 0.3 0.3; visual box size=0.3 0.3 0.3
- added link InertialWheel_1, mass 0.25; visual cylinder length=0.01 radius=0.08
- added link InertialWheel_2, mass 0.25; visual cylinder length=0.01 radius=0.08
- added link InertialWheel_3, mass 0.25; visual cylinder length=0.01 radius=0.08
- added link InertialWheel_4, mass 0.25; visual cylinder length=0.01 radius=0.08
- added link InertialWheel_5, mass 0.25; visual cylinder length=0.01 radius=0.08
- added link InertialWheel_6, mass 0.25; visual cylinder length=0.01 radius=0.08
Joints:
- added joint $continuous_CubeBody_InertialWheel_1: type continuous, parent CubeBody, child InertialWheel_1, origin xyz=0.15 0 0 rpy=0 1.57075 0, axis 0 0 1
- added joint $continuous_CubeBody_InertialWheel_2: type continuous, parent CubeBody, child InertialWheel_2, origin xyz=-0.15 0 0 rpy=0 1.57075 0, axis 0 0 1
- added joint $continuous_CubeBody_InertialWheel_3: type continuous, parent CubeBody, child InertialWheel_3, origin xyz=0 0.15 0 rpy=1.57075 0 0, axis 0 0 1
- added joint $continuous_CubeBody_InertialWheel_4: type continuous, parent CubeBody, child InertialWheel_4, origin xyz=0 -0.15 0 rpy=1.57075 0 0, axis 0 0 1
- added joint $continuous_CubeBody_InertialWheel_5: type continuous, parent CubeBody, child InertialWheel_5, origin xyz=0 0 0.15 rpy=0 0 1.57075, axis 0 0 1
- added joint $continuous_CubeBody_InertialWheel_6: type continuous, parent CubeBody, child InertialWheel_6, origin xyz=0 0 -0.15 rpy=0 0 1.57075, axis 0 0 1
- added joint $fixed_CubeBody_CornerBumper_1: type fixed, parent CubeBody, child CornerBumper_1, origin xyz=0.15 0.15 0.15 rpy=0 0 0
- added joint $fixed_CubeBody_CornerBumper_2: type fixed, parent CubeBody, child CornerBumper_2, origin xyz=-0.15 0.15 0.15 rpy=0 0 0
- added joint $fixed_CubeBody_CornerBumper_3: type fixed, parent CubeBody, child CornerBumper_3, origin xyz=0.15 -0.15 0.15 rpy=0 0 0
- added joint $fixed_CubeBody_CornerBumper_4: type fixed, parent CubeBody, child CornerBumper_4, origin xyz=-0.15 -0.15 0.15 rpy=0 0 0
- added joint $fixed_CubeBody_CornerBumper_5: type fixed, parent CubeBody, child CornerBumper_5, origin xyz=0.15 0.15 -0.15 rpy=0 0 0
- added joint $fixed_CubeBody_CornerBumper_6: type fixed, parent CubeBody, child CornerBumper_6, origin xyz=-0.15 0.15 -0.15 rpy=0 0 0
- added joint $fixed_CubeBody_CornerBumper_7: type fixed, parent CubeBody, child CornerBumper_7, origin xyz=0.15 -0.15 -0.15 rpy=0 0 0
- added joint $fixed_CubeBody_CornerBumper_8: type fixed, parent CubeBody, child CornerBumper_8, origin xyz=-0.15 -0.15 -0.15 rpy=0 0 0
